File: Hardware_KICAD/Raspbery_pi/Raspbery_pi.kicad_sch (KiCad schematic)
At the start: 8 parts, among them J1 Raspberry_Pi_2_3, J2 Conn_01x07_Socket, J3 Raspberry Pi Micro USB Power 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, SW1 MODE BUTTON, SW2 ACTION BUTTON, U1 BME680

Commit message: added report stuff
Parts:
- renumbered J2 to DS1
Changed lines of the file:
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@@
 		(on_board yes)
 		(dnp no)
-		(fields_autoplaced yes)
-		(property "Reference" "J2"
-			(at 70.485 105.41 0)
+		(property "Reference" "DS1"
+			(at 77.47 105.156 0)
 			(effects
 				(font
@@
 		)
 		(property "Value" "Conn_01x07_Socket"
-			(at 70.485 107.95 0)
+			(at 77.47 107.696 0)
 			(effects
 				(font
@@
 			(project ""
 				(path "/0b055c2c-172e-477e-bdb2-5c3199ca2401"
-					(reference "J2")
+					(reference "DS1")
 					(unit 1)
 				)
