File: Hardware_KICAD/GeekGoggles_Schematic/_autosave-voltmeter.kicad_sch (KiCad schematic)
At the start: 6 parts, among them J1 USB_B_Micro, SW3 SW_Push, U2 ESP32-S3-WROOM-1

Commit message: Merge_1
Connections:
- net 3.3V_ESP: now reaches U2.2 (3V3)
Other:
- moved on the sheet: D1, J1, R1, R2, SW3, U2
